Commit message: update files to fit with aroco parameters

File: robucar_description/urdf/robucar.urdf.xacro (robot description, xacro)
@@ -4,6 +4,6 @@
   <xacro:arg name="mode" default="simulation" />
   <xacro:arg name="controller_conf_yaml_file" default=""/>
-  <xacro:include filename="$(find adap2e_description)/urdf/robucar.xacro" />
-  <xacro:adap2e model="slim" mode="$(arg mode)" prefix="$(arg prefix)"/>
+  <xacro:include filename="$(find robucar_description)/urdf/robucar.xacro" />
+  <xacro:robucar mode="$(arg mode)" prefix="$(arg prefix)"/>
   <gazebo>
     <plugin filename="libgazebo_ros2_control.so" name="gazebo_ros2_control">

File: robucar_description/urdf/robucar.xacro (robot description, xacro)
@@ -1,84 +1,86 @@
 <?xml version="1.0"?>
-<robot name="adap2e" xmlns:xacro="http://www.ros.org/wiki/xacro">
-    <xacro:macro name="adap2e" params="model mode prefix">
-      <xacro:include filename="$(find romea_mobile_base_description)/urdf/4WS_4WD_chassis.xacro" />
-      <xacro:include filename="$(find romea_mobile_base_description)/ros2_control/4WS_4WD.ros2_control.xacro"/>
-      <xacro:property name="conf" value="$(find adap2e_description)/config/adap2e_${model}.yaml" />
-      <xacro:property name="props" value="${load_yaml(conf)['/**']['ros__parameters']['base_info']}" />
-      <!-- Link names -->
-      <xacro:property name="base_link" value="${props['links']['base_link_name']}" />
-      <xacro:property name="base_footprint_link" value="${props['links']['base_footprint_link_name']}" />
-      <xacro:property name="inertial_link" value="${props['links']['inertial_link_name']}" />
-      <xacro:property name="front_left_wheel_steering_link" value="${props['links']['front_left_wheel_steering_link_name']}" />
-      <xacro:property name="front_right_wheel_steering_link" value="${props['links']['front_right_wheel_steering_link_name']}" />
-      <xacro:property name="rear_left_wheel_steering_link" value="${props['links']['rear_left_wheel_steering_link_name']}" />
-      <xacro:property name="rear_right_wheel_steering_link" value="${props['links']['rear_right_wheel_steering_link_name']}" />
-      <xacro:property name="front_left_wheel_spinning_link" value="${props['links']['front_left_wheel_spinning_link_name']}" />
-      <xacro:property name="front_right_wheel_spinning_link" value="${props['links']['front_right_wheel_spinning_link_name']}" />
-      <xacro:property name="rear_left_wheel_spinning_link" value="${props['links']['rear_left_wheel_spinning_link_name']}" />
-      <xacro:property name="rear_right_wheel_spinning_link" value="${props['links']['rear_right_wheel_spinning_link_name']}" />
-      <!-- Joint names -->
-      <xacro:property name="base_footprint_joint" value="${props['joints']['base_footprint_joint_name']}" />
-      <xacro:property name="inertial_joint" value="${props['joints']['inertial_joint_name']}" />
-      <xacro:property name="front_left_wheel_steering_joint" value="${props['joints']['front_left_wheel_steering_joint_name']}" />
-      <xacro:property name="front_right_wheel_steering_joint" value="${props['joints']['front_right_wheel_steering_joint_name']}" />
-      <xacro:property name="rear_left_wheel_steering_joint" value="${props['joints']['rear_left_wheel_steering_joint_name']}" />
-      <xacro:property name="rear_right_wheel_steering_joint" value="${props['joints']['rear_right_wheel_steering_joint_name']}" />
-      <xacro:property name="front_left_wheel_spinning_joint" value="${props['joints']['front_left_wheel_spinning_joint_name']}" />
-      <xacro:property name="front_right_wheel_spinning_joint" value="${props['joints']['front_right_wheel_spinning_joint_name']}" />
-      <xacro:property name="rear_left_wheel_spinning_joint" value="${props['joints']['rear_left_wheel_spinning_joint_name']}" />
-      <xacro:property name="rear_right_wheel_spinning_joint" value="${props['joints']['rear_right_wheel_spinning_joint_name']}" />
-      <!-- Base Properties -->
-      <xacro:property name="aabb_length" value="${props['geometry']['aabb']['length']}" />
-      <xacro:property name="aabb_width" value="${props['geometry']['aabb']['width']}" />
-      <xacro:property name="aabb_height" value="${props['geometry']['aabb']['height']}" />
-      <xacro:property name="wheelbase" value="${props['geometry']['axles_distance']}"/>
-      <xacro:property name="front_track" value="${props['geometry']['front_axle']['wheels_distance']}"/>
-      <xacro:property name="rear_track" value="${props['geometry']['rear_axle']['wheels_distance']}"/>
-      <xacro:property name="mass_base" value="${props['inertia']['mass']}" />
-      <xacro:property name="mass_center_x" value="${props['inertia']['center'][0]}" />
-      <xacro:property name="mass_center_y" value="${props['inertia']['center'][1]}" />
-      <xacro:property name="mass_center_z" value="${props['inertia']['center'][2]}" />
-      <xacro:property name="minimal_wheel_steering_angle" value="-${props['wheels_steering_control']['command']['maximal_angle']}"/>
-      <xacro:property name="maximal_wheel_steering_angle" value="${props['wheels_steering_control']['command']['maximal_angle']}"/>
-      <xacro:property name="maximal_wheel_speed" value="${props['wheels_speed_control']['command']['maximal_speed']}"/>
-      <xacro:property name="body_reference_x" value="${props['control_point'][0]}" />
-      <!-- Wheel Properties -->
-      <xacro:property name="steering_link_mass" value="3" />
-      <xacro:property name="steering_link_y" value="0.05" />
-      <xacro:property name="steering_link_xz" value="0.1" />
-      <xacro:property name="front_wheel_radius" value="${props['geometry']['front_axle']['wheels']['radius']}" />
-      <xacro:property name="rear_wheel_radius" value="${props['geometry']['rear_axle']['wheels']['radius']}" />
-      <xacro:property name="front_wheel_width" value="${props['geometry']['front_axle']['wheels']['width']}" />
-      <xacro:property name="rear_wheel_width" value="${props['geometry']['rear_axle']['wheels']['width']}" />
-      <xacro:property name="front_wheel_mass" value="10" />
-      <xacro:property name="rear_wheel_mass" value="10" />
-      <!-- Wheel Mounting Positions -->
-      <xacro:property name="ground_clearance" value="${props['geometry']['ground_clearance']}"/>
-      <xacro:property name="front_wheel_y_offset" value="${props['geometry']['front_axle']['wheels']['hub_carrier_offset']}" />
-      <xacro:property name="rear_wheel_y_offset" value="${props['geometry']['rear_axle']['wheels']['hub_carrier_offset']}" />
-      <xacro:property name="chassis_height" value="${min(front_wheel_radius,rear_wheel_radius)}" />
-      <!-- Ros2 control hardware plugin -->
-      <xacro:property name="simulation_hardware_plugin" value="romea_mobile_base_gazebo/GazeboSystemInterface4WS4WD"/>
-      <xacro:property name="live_hardware_plugin" value="adap2e_hardware/Adap2eHardware"/>
-      <!-- visual chassis -->
+<robot name="robucar" xmlns:xacro="http://www.ros.org/wiki/xacro">
+    <xacro:include filename="$(find romea_mobile_base_description)/urdf/2AS_4WD_chassis.xacro" />
+    <xacro:include filename="$(find romea_mobile_base_description)/ros2_control/2AS_4WD.ros2_control.xacro"/>
+    <xacro:property name="conf" value="$(find robucar_description)/config/robucar.yaml" />
+    <xacro:property name="props" value="${load_yaml(conf)['/**']['ros__parameters']['base_info']}" />
+    <!-- Link names -->
+    <xacro:property name="base_link" value="${props['links']['base_link_name']}" />
+    <xacro:property name="base_footprint_link" value="${props['links']['base_footprint_link_name']}" />
+    <xacro:property name="inertial_link" value="${props['links']['inertial_link_name']}" />
+    <xacro:property name="front_axle_steering_link" value="${props['links']['front_axle_steering_link_name']}" />
+    <xacro:property name="rear_axle_steering_link" value="${props['links']['rear_axle_steering_link_name']}" />
+    <xacro:property name="front_left_wheel_steering_link" value="${props['links']['front_left_wheel_steering_link_name']}" />
+    <xacro:property name="front_right_wheel_steering_link" value="${props['links']['front_right_wheel_steering_link_name']}" />
+    <xacro:property name="rear_left_wheel_steering_link" value="${props['links']['rear_left_wheel_steering_link_name']}" />
+    <xacro:property name="rear_right_wheel_steering_link" value="${props['links']['rear_right_wheel_steering_link_name']}" />
+    <xacro:property name="front_left_wheel_spinning_link" value="${props['links']['front_left_wheel_spinning_link_name']}" />
+    <xacro:property name="front_right_wheel_spinning_link" value="${props['links']['front_right_wheel_spinning_link_name']}" />
+    <xacro:property name="rear_left_wheel_spinning_link" value="${props['links']['rear_left_wheel_spinning_link_name']}" />
+    <xacro:property name="rear_right_wheel_spinning_link" value="${props['links']['rear_right_wheel_spinning_link_name']}" />
+    <!-- Joint names -->
+    <xacro:property name="base_footprint_joint" value="${props['joints']['base_footprint_joint_name']}" />
+    <xacro:property name="inertial_joint" value="${props['joints']['inertial_joint_name']}" />
+    <xacro:property name="front_axle_steering_joint" value="${props['joints']['front_axle_steering_joint_name']}" />
+    <xacro:property name="rear_axle_steering_joint" value="${props['joints']['rear_axle_steering_joint_name']}" />
+    <xacro:property name="front_left_wheel_steering_joint" value="${props['joints']['front_left_wheel_steering_joint_name']}" />
+    <xacro:property name="front_right_wheel_steering_joint" value="${props['joints']['front_right_wheel_steering_joint_name']}" />
+    <xacro:property name="rear_left_wheel_steering_joint" value="${props['joints']['rear_left_wheel_steering_joint_name']}" />
+    <xacro:property name="rear_right_wheel_steering_joint" value="${props['joints']['rear_right_wheel_steering_joint_name']}" />
+    <xacro:property name="front_left_wheel_spinning_joint" value="${props['joints']['front_left_wheel_spinning_joint_name']}" />
+    <xacro:property name="front_right_wheel_spinning_joint" value="${props['joints']['front_right_wheel_spinning_joint_name']}" />
+    <xacro:property name="rear_left_wheel_spinning_joint" value="${props['joints']['rear_left_wheel_spinning_joint_name']}" />
+    <xacro:property name="rear_right_wheel_spinning_joint" value="${props['joints']['rear_right_wheel_spinning_joint_name']}" />
+    <!-- Base Properties -->
+    <xacro:property name="aabb_length" value="${props['geometry']['aabb']['length']}" />
+    <xacro:property name="aabb_width" value="${props['geometry']['aabb']['width']}" />
+    <xacro:property name="aabb_height" value="${props['geometry']['aabb']['height']}" />
+    <xacro:property name="wheelbase" value="${props['geometry']['axles_distance']}"/>
+    <xacro:property name="front_track" value="${props['geometry']['front_axle']['wheels_distance']}"/>
+    <xacro:property name="rear_track" value="${props['geometry']['rear_axle']['wheels_distance']}"/>
+    <xacro:property name="mass_base" value="${props['inertia']['mass']}" />
+    <xacro:property name="mass_center_x" value="${props['inertia']['center'][0]}" />
+    <xacro:property name="mass_center_y" value="${props['inertia']['center'][1]}" />
+    <xacro:property name="mass_center_z" value="${props['inertia']['center'][2]}" />
+    <xacro:property name="maximal_axle_steering_angle" value="${props['axles_steering_control']['command']['maximal_angle']}"/>
+    <xacro:property name="maximal_wheel_steering_angle" value="${atan(tan(maximal_axle_steering_angle)/(1-tan(maximal_axle_steering_angle)*front_track/(2*wheelbase)))}"/>
+    <xacro:property name="minimal_axle_steering_angle" value="${-maximal_axle_steering_angle}"/>
+    <xacro:property name="minimal_wheel_steering_angle" value="${-maximal_wheel_steering_angle} "/>
+    <xacro:property name="maximal_wheel_speed" value="${props['wheels_speed_control']['command']['maximal_speed']}"/>
+    <xacro:property name="body_reference_x" value="${props['control_point'][0]}" />
+    <!-- Wheel Properties -->
+    <xacro:property name="steering_link_mass" value="3" />
+    <xacro:property name="steering_link_y" value="0.05" />
+    <xacro:property name="steering_link_xz" value="0.1" />
+    <xacro:property name="front_wheel_radius" value="${props['geometry']['front_axle']['wheels']['radius']}" />
+    <xacro:property name="rear_wheel_radius" value="${props['geometry']['rear_axle']['wheels']['radius']}" />
+    <xacro:property name="front_wheel_width" value="${props['geometry']['front_axle']['wheels']['width']}" />
+    <xacro:property name="rear_wheel_width" value="${props['geometry']['rear_axle']['wheels']['width']}" />
+    <xacro:property name="front_wheel_mass" value="10" />
+    <xacro:property name="rear_wheel_mass" value="10" />
+    <!-- Wheel Mounting Positions -->
+    <xacro:property name="ground_clearance" value="${props['geometry']['ground_clearance']}"/>
+    <xacro:property name="front_wheel_y_offset" value="${props['geometry']['front_axle']['wheels']['hub_carrier_offset']}" />
+    <xacro:property name="rear_wheel_y_offset" value="${props['geometry']['rear_axle']['wheels']['hub_carrier_offset']}" />
+    <xacro:property name="chassis_height" value="${min(front_wheel_radius,rear_wheel_radius)}" />
+    <!-- Ros2 control hardware plugin -->
+    <xacro:property name="simulation_hardware_plugin" value="romea_mobile_base_gazebo/GazeboSystemInterface2AS4WD"/>
+    <xacro:property name="live_hardware_plugin" value="robucar_hardware/RobucarHardware"/>
+    <xacro:macro name="robucar" params="mode prefix">
       <xacro:chassis>
-         <visual>
-           <origin xyz="${-body_reference_x} 0 ${chassis_height}" rpy="0 0 ${M_PI/2.0}" />
-           <geometry>
-             <mesh filename="package://adap2e_description/meshes/framev3_05.dae"/>
-           </geometry>
-           <material name="grey">
-             <color rgba="0.6 0.6 0.6 1"/>
-           </material>
+        <visual>
+          <origin xyz="${-body_reference_x} 0 ${chassis_height-aabb_height/2}" rpy="0 0 ${M_PI/2.0}" />
+          <geometry>
+            <mesh filename="package://robucar_description/meshes/chassis.dae"/>
+          </geometry>
         </visual>
-        <!-- steering geometry -->
-        <box size="0.05 ${steering_link_y} 0.05"/>
-        <!-- wheel geometry -->
-        <mesh filename="package://adap2e_description/meshes/wheel_02.dae"/>
+        <!-- visual steering -->
+        <mesh filename="package://robucar_description/meshes/wheel_steered.dae"/>
+        <!-- visual wheel -->
+        <mesh filename="package://robucar_description/meshes/wheel.dae"/>
       </xacro:chassis>
-     <xacro:if value="${mode == 'simulation' or mode == 'live'}">
-        <xacro:base_control mode="${mode}"/>
-     </xacro:if>
-  </xacro:macro>
+      <xacro:if value="${mode == 'simulation' or mode == 'live'}">
+         <xacro:base_control mode="${mode}"/>
+      </xacro:if>
+    </xacro:macro>
 </robot>

Commit message: split ros2_control from urdf remove robot state publisher

File: robucar_description/urdf/robucar.urdf.xacro (robot description, xacro)
@@ -3,15 +3,16 @@
   <xacro:arg name="prefix" default="robucar_" />
   <xacro:arg name="mode" default="simulation" />
-  <xacro:arg name="controller_conf_yaml_file" default="" />
+  <xacro:arg name="base_name" default="base" />
+  <xacro:arg name="ros2_control_config_urdf_file" default="" />
+  <xacro:arg name="controller_manager_config_yaml_file" default="" />
   <xacro:arg name="ros_prefix" default="/robufast/" />
   <xacro:include filename="$(find robucar_description)/urdf/robucar.xacro" />
   <xacro:robucar mode="$(arg mode)" prefix="$(arg prefix)" />
   <gazebo>
-    <plugin filename="libgazebo_ros2_control.so" name="gazebo_ros2_control">
-      <hardware>$(arg prefix)base</hardware>
-      <robot_param_node>$(arg ros_prefix)robot_state_publisher</robot_param_node>
-      <parameters>$(arg controller_conf_yaml_file)</parameters>
+    <plugin filename="libromea_gazebo_ros2_control.so" name="gazebo_ros2_control">
+      <ros2_control_config_file>$(arg ros2_control_config_urdf_file)</ros2_control_config_file>
+      <controller_manager_config_file>$(arg controller_manager_config_yaml_file)</controller_manager_config_file>
       <ros>
-        <namespace>$(arg ros_prefix)base</namespace>
+        <namespace>$(arg ros_prefix)$(arg base_name)</namespace>
       </ros>
     </plugin>

File: robucar_description/urdf/robucar.xacro (robot description, xacro)
@@ -2,6 +2,4 @@
 <robot name="robucar" xmlns:xacro="http://www.ros.org/wiki/xacro">
   <xacro:include filename="$(find romea_mobile_base_description)/urdf/base2ASxxx.chassis.xacro" />
-  <xacro:include
-    filename="$(find romea_mobile_base_description)/ros2_control/base2AS4WD.ros2_control.xacro" />
   <xacro:property name="conf" value="$(find robucar_description)/config/robucar.yaml" />
   <xacro:property name="props" value="${load_yaml(conf)}" />
@@ -98,8 +96,4 @@
     value="${props['geometry']['rear_axle']['wheels']['hub_carrier_offset']}" />
   <xacro:property name="chassis_height" value="${min(front_wheel_radius,rear_wheel_radius)}" />
-  <!-- Ros2 control hardware plugin -->
-  <xacro:property name="simulation_hardware_plugin"
-    value="romea_mobile_base_gazebo/GazeboSystemInterface2AS4WD" />
-  <xacro:property name="live_hardware_plugin" value="robucar_hardware/RobucarHardware" />
   <xacro:macro name="robucar" params="mode prefix">
     <xacro:chassis>
@@ -115,7 +109,4 @@
       <mesh filename="package://robucar_description/meshes/wheel.dae" />
     </xacro:chassis>
-    <xacro:if value="${mode == 'simulation' or mode == 'live'}">
-      <xacro:base_control mode="${mode}" />
-    </xacro:if>
   </xacro:macro>
 </robot>
