Commit message: description:  add missing properties into ros2_control xacro file
Signed-off-by: jean.laneurit <jean.laneurit@inrae.fr>

File: robucar_description/ros2_control/robucar.ros2_control.xacro (robot description, xacro)
@@ -38,4 +38,8 @@
     <xacro:property name="rear_wheel_radius"
       value="${props['geometry']['rear_axle']['wheels']['radius']}" />
+    <xacro:property name="maximal_axle_steering_angle"
+      value="${props['axles_steering_control']['command']['maximal_angle']}" />
+    <xacro:property name="maximal_wheel_speed"
+      value="${props['wheels_speed_control']['command']['maximal_speed']}" />
     <!-- simulation plugins -->
     <xacro:property name="simulation_hardware_plugin"

Commit message: add compute maximal_wheel_steering_angle in ros2 control xacro file
Signed-off-by: jean.laneurit <jean.laneurit@inrae.fr>

File: robucar_description/ros2_control/robucar.ros2_control.xacro (robot description, xacro)
@@ -40,4 +40,6 @@
     <xacro:property name="maximal_axle_steering_angle"
       value="${props['axles_steering_control']['command']['maximal_angle']}" />
+    <xacro:property name="maximal_wheel_steering_angle"
+      value="${atan(tan(maximal_axle_steering_angle)/(1-tan(maximal_axle_steering_angle)*front_track/(2*wheelbase)))}" />
     <xacro:property name="maximal_wheel_speed"
       value="${props['wheels_speed_control']['command']['maximal_speed']}" />
