Commit message: [description] update ros2 control xacro file
Signed-off-by: Jean Laneurit <jean.laneurit@inrae.fr>

File: robucar_description/ros2_control/robucar.ros2_control.xacro (robot description, xacro)
@@ -44,10 +44,28 @@
     <xacro:property name="maximal_wheel_speed"
       value="${props['wheels_speed_control']['command']['maximal_speed']}" />
-    <!-- simulation plugins -->
-    <xacro:property name="simulation_hardware_plugin"
-      value="romea_mobile_base_gazebo/GazeboSystemInterface2AS4WD" />
-    <xacro:property name="live_hardware_plugin"
-      value="robucar_hardware/RobucarHardware" />
-    <xacro:base_control mode="${mode}" base_name="${base_name}" />
+    <xacro:if value="${mode == 'simulation_gazebo'}">
+      <xacro:property
+        name="hardware_plugin"
+        value="romea_mobile_base_gazebo/GazeboSystemInterface" />
+    </xacro:if>
+    <xacro:if value="${mode == 'simulation_gazebo_classic'}">
+      <xacro:property
+        name="hardware_plugin"
+        value="romea_mobile_base_gazebo/GazeboSystemInterface2AS4WD" />
+    </xacro:if>
+    <xacro:if value="${'4dv' in mode or 'isaac' in mode}">
+      <xacro:property
+        name="hardware_plugin"
+        value="romea_mobile_base_simulation/GenericSimulationSystemInterface" />
+    </xacro:if>
+    <xacro:if value="${mode ==  'live'}">
+      <xacro:property
+        name="hardware_plugin"
+        value="robucar_hardware/robucar_hardware" />
+    </xacro:if>
+    <xacro:base_control
+      mode="${mode}"
+      base_name="${base_name}"
+      hardware_plugin="${hardware_plugin}" />
   </xacro:macro>
 </robot>

Commit message: [description] add robcar_properties.xacro
Signed-off-by: Jean Laneurit <jean.laneurit@inrae.fr>

File: robucar_description/ros2_control/robucar.ros2_control.xacro (robot description, xacro)
@@ -5,43 +5,5 @@
       filename="$(find romea_mobile_base_description)/ros2_control/base2AS4WD.ros2_control.xacro" />
     <xacro:property name="conf" value="$(find robucar_description)/config/robucar.yaml" />
-    <xacro:property name="props" value="${load_yaml(conf)}" />
-    <!-- Joint names -->
-    <xacro:property name="front_axle_steering_joint"
-      value="${props['joints']['front_axle_steering_joint_name']}" />
-    <xacro:property name="rear_axle_steering_joint"
-      value="${props['joints']['rear_axle_steering_joint_name']}" />
-    <xacro:property name="front_left_wheel_steering_joint"
-      value="${props['joints']['front_left_wheel_steering_joint_name']}" />
-    <xacro:property name="front_right_wheel_steering_joint"
-      value="${props['joints']['front_right_wheel_steering_joint_name']}" />
-    <xacro:property name="rear_left_wheel_steering_joint"
-      value="${props['joints']['rear_left_wheel_steering_joint_name']}" />
-    <xacro:property name="rear_right_wheel_steering_joint"
-      value="${props['joints']['rear_right_wheel_steering_joint_name']}" />
-    <xacro:property name="front_left_wheel_spinning_joint"
-      value="${props['joints']['front_left_wheel_spinning_joint_name']}" />
-    <xacro:property name="front_right_wheel_spinning_joint"
-      value="${props['joints']['front_right_wheel_spinning_joint_name']}" />
-    <xacro:property name="rear_left_wheel_spinning_joint"
-      value="${props['joints']['rear_left_wheel_spinning_joint_name']}" />
-    <xacro:property name="rear_right_wheel_spinning_joint"
-      value="${props['joints']['rear_right_wheel_spinning_joint_name']}" />
-    <!-- Geometry -->
-    <xacro:property name="wheelbase"
-      value="${props['geometry']['axles_distance']}" />
-    <xacro:property name="front_track"
-      value="${props['geometry']['front_axle']['wheels_distance']}" />
-    <xacro:property name="rear_track"
-      value="${props['geometry']['rear_axle']['wheels_distance']}" />
-    <xacro:property name="front_wheel_radius"
-      value="${props['geometry']['front_axle']['wheels']['radius']}" />
-    <xacro:property name="rear_wheel_radius"
-      value="${props['geometry']['rear_axle']['wheels']['radius']}" />
-    <xacro:property name="maximal_axle_steering_angle"
-      value="${props['axles_steering_control']['command']['maximal_angle']}" />
-    <xacro:property name="maximal_wheel_steering_angle"
-      value="${atan(tan(maximal_axle_steering_angle)/(1-tan(maximal_axle_steering_angle)*front_track/(2*wheelbase)))}" />
-    <xacro:property name="maximal_wheel_speed"
-      value="${props['wheels_speed_control']['command']['maximal_speed']}" />
+    <xacro:include filename="$(find robucar_description)/urdf/robucar_properties.xacro" />
     <xacro:if value="${mode == 'simulation_gazebo'}">
       <xacro:property

File: robucar_description/urdf/robucar.xacro (robot description, xacro)
@@ -6,124 +6,5 @@
   <xacro:include filename="$(find robucar_description)/urdf/visual/arms.xacro" />
   <xacro:property name="conf" value="$(find robucar_description)/config/robucar.yaml" />
-  <xacro:property name="props" value="${load_yaml(conf)}" />
-  <!-- Link names -->
-  <xacro:property name="base_link" value="${props['links']['base_link_name']}" />
-  <xacro:property name="base_footprint_link" value="${props['links']['base_footprint_link_name']}" />
-  <xacro:property name="inertial_link" value="${props['links']['inertial_link_name']}" />
-  <xacro:property name="front_axle_steering_link"
-    value="${props['links']['front_axle_steering_link_name']}" />
-  <xacro:property name="rear_axle_steering_link"
-    value="${props['links']['rear_axle_steering_link_name']}" />
-  <xacro:property name="front_left_wheel_steering_link"
-    value="${props['links']['front_left_wheel_steering_link_name']}" />
-  <xacro:property name="front_right_wheel_steering_link"
-    value="${props['links']['front_right_wheel_steering_link_name']}" />
-  <xacro:property name="rear_left_wheel_steering_link"
-    value="${props['links']['rear_left_wheel_steering_link_name']}" />
-  <xacro:property name="rear_right_wheel_steering_link"
-    value="${props['links']['rear_right_wheel_steering_link_name']}" />
-  <xacro:property name="front_left_wheel_spinning_link"
-    value="${props['links']['front_left_wheel_spinning_link_name']}" />
-  <xacro:property name="front_right_wheel_spinning_link"
-    value="${props['links']['front_right_wheel_spinning_link_name']}" />
-  <xacro:property name="rear_left_wheel_spinning_link"
-    value="${props['links']['rear_left_wheel_spinning_link_name']}" />
-  <xacro:property name="rear_right_wheel_spinning_link"
-    value="${props['links']['rear_right_wheel_spinning_link_name']}" />
-  <!-- Joint names -->
-  <xacro:property name="base_footprint_joint"
-    value="${props['joints']['base_footprint_joint_name']}" />
-  <xacro:property name="inertial_joint" value="${props['joints']['inertial_joint_name']}" />
-  <xacro:property name="front_axle_steering_joint"
-    value="${props['joints']['front_axle_steering_joint_name']}" />
-  <xacro:property name="rear_axle_steering_joint"
-    value="${props['joints']['rear_axle_steering_joint_name']}" />
-  <xacro:property name="front_left_wheel_steering_joint"
-    value="${props['joints']['front_left_wheel_steering_joint_name']}" />
-  <xacro:property name="front_right_wheel_steering_joint"
-    value="${props['joints']['front_right_wheel_steering_joint_name']}" />
-  <xacro:property name="rear_left_wheel_steering_joint"
-    value="${props['joints']['rear_left_wheel_steering_joint_name']}" />
-  <xacro:property name="rear_right_wheel_steering_joint"
-    value="${props['joints']['rear_right_wheel_steering_joint_name']}" />
-  <xacro:property name="front_left_wheel_spinning_joint"
-    value="${props['joints']['front_left_wheel_spinning_joint_name']}" />
-  <xacro:property name="front_right_wheel_spinning_joint"
-    value="${props['joints']['front_right_wheel_spinning_joint_name']}" />
-  <xacro:property name="rear_left_wheel_spinning_joint"
-    value="${props['joints']['rear_left_wheel_spinning_joint_name']}" />
-  <xacro:property name="rear_right_wheel_spinning_joint"
-    value="${props['joints']['rear_right_wheel_spinning_joint_name']}" />
-  <!-- Base Properties -->
-  <xacro:property name="aabb_length"
-    value="${props['geometry']['aabb']['length']}" />
-  <xacro:property name="aabb_width"
-    value="${props['geometry']['aabb']['width']}" />
-  <xacro:property name="aabb_height"
-    value="${props['geometry']['aabb']['height']}" />
-  <xacro:property name="aabb_center_x"
-    value="${props['geometry']['aabb']['center'][0]}" />
-  <xacro:property name="aabb_center_y"
-    value="${props['geometry']['aabb']['center'][1]}" />
-  <xacro:property name="aabb_center_z"
-    value="${props['geometry']['aabb']['center'][2]}" />
-  <xacro:property name="wheelbase"
-    value="${props['geometry']['axles_distance']}" />
-  <xacro:property name="front_track"
-    value="${props['geometry']['front_axle']['wheels_distance']}" />
-  <xacro:property name="rear_track"
-    value="${props['geometry']['rear_axle']['wheels_distance']}" />
-  <xacro:property name="mass_base"
-    value="${props['inertia']['mass']}" />
-  <xacro:property name="mass_center_x"
-    value="${props['inertia']['center'][0]}" />
-  <xacro:property name="mass_center_y"
-    value="${props['inertia']['center'][1]}" />
-  <xacro:property name="mass_center_z"
-    value="${props['inertia']['center'][2]}" />
-  <xacro:property name="body_reference_x"
-    value="${props['control_point'][0]}" />
-  <xacro:property name="ground_clearance"
-    value="${props['geometry']['ground_clearance']}" />
-  <!-- Wheel Properties -->
-  <xacro:property name="front_wheel_x_offset" value="0.0" />
-  <xacro:property name="rear_wheel_x_offset" value="0.0" />
-  <xacro:property name="front_hub_carrier_offset"
-    value="${props['geometry']['front_axle']['wheels']['hub_carrier_offset']}" />
-  <xacro:property name="rear_hub_carrier_offset"
-    value="${props['geometry']['rear_axle']['wheels']['hub_carrier_offset']}" />
-  <xacro:property name="front_wheel_radius"
-    value="${props['geometry']['front_axle']['wheels']['radius']}" />
-  <xacro:property name="rear_wheel_radius"
-    value="${props['geometry']['rear_axle']['wheels']['radius']}" />
-  <xacro:property name="front_wheel_width"
-    value="${props['geometry']['front_axle']['wheels']['width']}" />
-  <xacro:property name="rear_wheel_width"
-    value="${props['geometry']['rear_axle']['wheels']['width']}" />
-  <xacro:property name="chassis_height"
-    value="${min(front_wheel_radius,rear_wheel_radius)}" />
-  <xacro:property name="maximal_wheel_speed"
-    value="${props['wheels_speed_control']['command']['maximal_speed']}" />
-  <xacro:property name="front_wheel_mass" value="10" />
-  <xacro:property name="rear_wheel_mass" value="10" />
-  <!-- Steering Properties -->
-  <xacro:property name="maximal_axle_steering_angle"
-    value="${props['axles_steering_control']['command']['maximal_angle']}" />
-  <xacro:property name="maximal_wheel_steering_angle"
-    value="${atan(tan(maximal_axle_steering_angle)/(1-tan(maximal_axle_steering_angle)*front_track/(2*wheelbase)))}" />
-  <xacro:property name="minimal_axle_steering_angle"
-    value="${-maximal_axle_steering_angle}" />
-  <xacro:property name="minimal_wheel_steering_angle"
-    value="${-maximal_wheel_steering_angle}" />
-  <xacro:property name="front_axle_steering_link_mass" value="1" />
-  <xacro:property name="front_axle_steering_link_x" value="0.05" />
-  <xacro:property name="front_axle_steering_link_y" value="0.05" />
-  <xacro:property name="front_axle_steering_link_z" value="0.05" />
-  <xacro:property name="front_wheel_steering_link_mass" value="20" />
-  <xacro:property name="front_wheel_steering_link_y" value="${front_hub_carrier_offset}" />
-  <xacro:property name="front_wheel_steering_link_xz" value="0.05" />
-  <xacro:property name="rear_wheel_steering_link_mass" value="20" />
-  <xacro:property name="rear_wheel_steering_link_y" value="${rear_hub_carrier_offset}" />
-  <xacro:property name="rear_wheel_steering_link_xz" value="0.05" />
+  <xacro:include filename="$(find robucar_description)/urdf/robucar_properties.xacro" />
   <xacro:macro name="robucar" params="mode prefix">
     <xacro:chassis>
