Commit message: meta_bringup implementation
Signed-off-by: Jean Laneurit <jean.laneurit@inrae.fr>

File: robucar_description/ros2_control/robucar.ros2_control.urdf.xacro (robot description, xacro)
@@ -1,5 +1,5 @@
 <?xml version='1.0' encoding='utf-8'?>
 <robot name="robucar_ros2_control" xmlns:xacro="http://www.ros.org/wiki/xacro">
-  <xacro:arg name="prefix" default="aroco_" />
+  <xacro:arg name="prefix" default="robucar_" />
   <xacro:arg name="mode" default="simulation" />
   <xacro:arg name="base_name" default="base" />

File: robucar_description/urdf/robucar.urdf.xacro (robot description, xacro)
@@ -4,17 +4,13 @@
   <xacro:arg name="mode" default="simulation" />
   <xacro:arg name="base_name" default="base" />
-  <xacro:arg name="ros2_control_config_urdf_file" default="" />
   <xacro:arg name="controller_manager_config_yaml_file" default="" />
   <xacro:arg name="ros_prefix" default="/robufast/" />
   <xacro:include filename="$(find robucar_description)/urdf/robucar.xacro" />
   <xacro:robucar mode="$(arg mode)" prefix="$(arg prefix)" />
-  <gazebo>
-    <plugin filename="libromea_gazebo_ros2_control.so" name="gazebo_ros2_control">
-      <ros2_control_config_file>$(arg ros2_control_config_urdf_file)</ros2_control_config_file>
-      <controller_manager_config_file>$(arg controller_manager_config_yaml_file)</controller_manager_config_file>
-      <ros>
-        <namespace>$(arg ros_prefix)$(arg base_name)</namespace>
-      </ros>
-    </plugin>
-  </gazebo>
+  <xacro:include filename="$(find robucar_description)/urdf/robucar.simulation.xacro" />
+  <xacro:robucar_simulation
+    mode="$(arg mode)"
+    base_name="$(arg base_name)"
+    ros_prefix="$(arg ros_prefix)"
+    controller_manager_config_yaml_file="$(arg controller_manager_config_yaml_file)" />
 </robot>

File: robucar_description/urdf/visual/arms.xacro (robot description, xacro)
@@ -5,5 +5,6 @@
             <origin xyz="0.0 0.0 0.0" rpy="0 0 ${orientation}" />
             <geometry>
-                <mesh filename="package://robucar_description/meshes/wheel_steered.dae" />
+                <!-- <mesh filename="package://robucar_description/meshes/wheel_steered.dae" /> -->
+                <mesh filename="$(find robucar_description)/meshes/wheel_steered.dae" />
             </geometry>
             <material name=" grey">

File: robucar_description/urdf/visual/chassis.xacro (robot description, xacro)
@@ -6,5 +6,6 @@
                 rpy="0 0 ${M_PI/2.0}" />
             <geometry>
-                <mesh filename="package://robucar_description/meshes/chassis.dae" />
+                <!-- <mesh filename="package://robucar_description/meshes/chassis.dae" /> -->
+                <mesh filename="file://$(find robucar_description)/meshes/chassis.dae" />
             </geometry>
         </visual>

File: robucar_description/urdf/visual/wheels.xacro (robot description, xacro)
@@ -5,5 +5,6 @@
             <origin xyz="0 0 0" rpy="0 ${orientation} 0" />
             <geometry>
-                <mesh filename="package://robucar_description/meshes/wheel.dae" />
+                <!-- <mesh filename="package://robucar_description/meshes/wheel.dae" /> -->
+                <mesh filename="$(find robucar_description)/meshes/wheel.dae" />
             </geometry>
             <material name="black">
